File: BreakoutBoards/LED_RGB/LED_RGB.kicad_sch (KiCad schematic)
At the start: 6 parts, among them J1 Conn_01x04_Pin

Commit message: replaced out of stock resistors
Parts:
- removed R1, R2, R3: CR0603-FX-1001ELF, clectric-diy:R0603, symbol clectric-diy:CR0603-FX-1001ELF
- removed TP1: TestPoint, TestPoint:TestPoint_THTPad_D1.0mm_Drill0.5mm, symbol Connector:TestPoint
- added R1, R2, R3: FRC0603F1001TS, clectric-diy:R0603, symbol clectric-diy:FRC0603F1001TS
- J1: value Conn_01x04_Pin -> HDR-TH_4P-P2.54-V-M
Connections:
- net LED_BLUE: now also R3.1, R3.2
- net LED_GREEN: now also R2.1, R2.2
- net LED_RED: now also R1.1, R1.2
Other:
- title: ChargeForge LED_RGB -> Charge LED_RGB
